Commit message: Compiled version of code. WIP

File: urdf/test_diff_canopen_system.ros2_control.xacro (robot description, xacro)
@@ -1,5 +1,5 @@
 <?xml version="1.0"?>
 <robot xmlns:xacro="http://www.ros.org/wiki/xacro">
-    <xacro:macro name="canopen_ros2_control_test" params="
+    <xacro:macro name="diff_canopen_ros2_control_test" params="
       name
       prefix

File: urdf/test_diff_canopen_system.urdf.xacro (robot description, xacro)
@@ -8,6 +8,6 @@
     <xacro:arg name="master_bin" default=""/>
     <!-- ros2 control include -->
-    <xacro:include filename="$(find diff_canopen_system)/urdf/diff_canopen_system.ros2_control.xacro"/>
-    <xacro:canopen_ros2_control_test
+    <xacro:include filename="$(find diff_canopen_system)/urdf/test_diff_canopen_system.ros2_control.xacro"/>
+    <xacro:diff_canopen_ros2_control_test
       name="$(arg name)"
       prefix="$(arg prefix)"
