Commit message: set up mock hardware example launch file

File: urdf/mav1500.urdf.xacro (robot description, xacro)
@@ -9,11 +9,18 @@
     <!-- ros2 control include -->
     <xacro:include filename="$(find diff_canopen_system)/urdf/mav1500/mav1500_new.ros2_control.xacro"/>
+    <xacro:include filename="$(find diff_canopen_system)/urdf/mav1500/mav1500_plc.ros2_control.xacro"/>
     <xacro:mav1500_ros2_control
       name="$(arg name)"
       prefix="$(arg prefix)"
+      mock_hardware="true"
+      mock_sensor_commands="true"
       bus_config="$(arg bus_config)"
       master_config="$(arg master_config)"
       can_interface_name="$(arg can_interface_name)"
       master_bin="$(arg master_bin)"
+    />
+    <xacro:mav1500_plc_ros2_control
+      name="$(arg name)"
+      prefix="$(arg prefix)"
     />
     <link name="$(arg prefix)base_link"/>

File: urdf/mav1500/mav1500_new.ros2_control.xacro (robot description, xacro)
@@ -5,16 +5,24 @@
               name
               prefix
+              mock_hardware
+              mock_sensor_commands
               bus_config
               master_config
               can_interface_name
               master_bin">
-  <ros2_control name="${name}" type="system">
+  <ros2_control name="${name}_CANOPEN" type="system">
     <hardware>
-      <plugin>custom_mapping_canopen_system/CustomMappingCanopenSystem</plugin>
-      <param name="bus_config">${bus_config}</param>
-      <param name="master_config">${master_config}</param>
-      <param name="can_interface_name">${can_interface_name}</param>
-      <param name="master_bin">"${master_bin}"</param>
-      <param name="enable_canopen_interfaces">true</param>
+        <xacro:if value="${mock_hardware}">
+            <plugin>mock_components/GenericSystem</plugin>
+            <param name="mock_sensor_commands">${mock_sensor_commands}</param>
+        </xacro:if>
+        <xacro:unless value="${mock_hardware}">
+            <plugin>custom_mapping_canopen_system/CustomMappingCanopenSystem</plugin>
+            <param name="bus_config">${bus_config}</param>
+            <param name="master_config">${master_config}</param>
+            <param name="can_interface_name">${can_interface_name}</param>
+            <param name="master_bin">"${master_bin}"</param>
+            <param name="enable_canopen_interfaces">true</param>
+        </xacro:unless>
     </hardware>
     <joint name="${prefix}left_wheel">
@@ -26,5 +34,27 @@
       <xacro:dana_tm4_interfaces_mapping inverse_direction="false"/>
     </joint>
+    <sensor name="left_wheel">
+        <xacro:sensor_mapping/>
+    </sensor>
+    <sensor name="right_wheel">
+        <xacro:sensor_mapping/>
+    </sensor>
   </ros2_control>
+</xacro:macro>
+<xacro:macro name="sensor_mapping" params="inverse_direction:=false">
+    <state_interface name="battery_voltage" data_type="uint16_t">
+        <param name="data_type">uint16_t</param>
+        <param name="index">0x2124</param>
+        <param name="subindex">0x0</param>
+        <param name="unit">V</param>
+        <param name="from_hw_scaling_factor">0.01</param>
+    </state_interface>
+    <state_interface name="battery_current" data_type="int16_t">
+        <param name="data_type">int16_t</param>
+        <param name="index">0x2127</param>
+        <param name="subindex">0x0</param>
+        <param name="unit">A</param>
+        <param name="from_hw_scaling_factor">0.1</param>
+    </state_interface>
 </xacro:macro>
 <xacro:macro name="dana_tm4_interfaces_mapping" params="inverse_direction:=false">
@@ -39,6 +69,4 @@
   <command_interface name="drive_enable" data_type="bool">
     <param name="data_type">bool</param>
-    <param name="min">0</param>
-    <param name="max">1</param>
     <param name="index">0x2100</param>
     <param name="subindex">0x0</param>
@@ -46,6 +74,4 @@
   <command_interface name="main_contactor" data_type="bool">
     <param name="data_type">bool</param>
-    <param name="min">0</param>
-    <param name="max">1</param>
     <param name="index">0x2101</param>
     <param name="subindex">0x0</param>
@@ -53,6 +79,4 @@
   <command_interface name="break_release" data_type="bool">
     <param name="data_type">bool</param>
-    <param name="min">0</param>
-    <param name="max">1</param>
     <param name="index">0x2102</param>
     <param name="subindex">0x0</param>
@@ -60,6 +84,4 @@
   <command_interface name="safe_stop" data_type="bool">
     <param name="data_type">bool</param>
-    <param name="min">0</param>
-    <param name="max">1</param>
     <param name="index">0x2107</param>
     <param name="subindex">0x0</param>
@@ -67,6 +89,4 @@
   <command_interface name="control_mode" data_type="bool">
     <param name="data_type">bool</param>
-    <param name="min">0</param>
-    <param name="max">1</param>
     <param name="index">0x2108</param>
     <param name="subindex">0x0</param>
@@ -74,6 +94,4 @@
   <command_interface name="speed_control" data_type="bool">
     <param name="data_type">bool</param>
-    <param name="min">0</param>
-    <param name="max">1</param>
     <param name="index">0x2109</param>
     <param name="subindex">0x0</param>
@@ -81,6 +99,4 @@
   <command_interface name="reset_fault" data_type="bool">
     <param name="data_type">bool</param>
-    <param name="min">0</param>
-    <param name="max">1</param>
     <param name="index">0x210F</param>
     <param name="subindex">0x0</param>
@@ -88,6 +104,4 @@
   <command_interface name="velocity" data_type="int16_t">
     <param name="data_type">int16_t</param>
-    <param name="min">-8000</param>
-    <param name="max">8000</param>
     <param name="index">0x2110</param>
     <param name="subindex">0x0</param>
@@ -97,6 +111,4 @@
   <command_interface name="torque" data_type="int16_t">
     <param name="data_type">int16_t</param>
-    <param name="min">-32768</param>
-    <param name="max">32767</param>
     <param name="index">0x2111</param>
     <param name="subindex">0x0</param>
@@ -106,6 +118,4 @@
   <state_interface name="power_stage_active" data_type="bool">
     <param name="data_type">bool</param>
-    <param name="min">0</param>
-    <param name="max">1</param>
     <param name="index">0x2114</param>
     <param name="subindex">0x0</param>
@@ -113,6 +123,4 @@
   <state_interface name="fault" data_type="bool">
     <param name="data_type">bool</param>
-    <param name="min">0</param>
-    <param name="max">1</param>
     <param name="index">0x2115</param>
     <param name="subindex">0x0</param>
@@ -120,6 +128,4 @@
   <state_interface name="torque_mode" data_type="bool">
     <param name="data_type">bool</param>
-    <param name="min">0</param>
-    <param name="max">1</param>
     <param name="index">0x2116</param>
     <param name="subindex">0x0</param>
@@ -127,6 +133,4 @@
   <state_interface name="main_contactor_status" data_type="bool">
     <param name="data_type">bool</param>
-    <param name="min">0</param>
-    <param name="max">1</param>
     <param name="index">0x2117</param>
     <param name="subindex">0x0</param>
@@ -134,6 +138,4 @@
   <state_interface name="can_enable" data_type="bool">
     <param name="data_type">bool</param>
-    <param name="min">0</param>
-    <param name="max">1</param>
     <param name="index">0x2118</param>
     <param name="subindex">0x0</param>
@@ -141,6 +143,4 @@
   <state_interface name="safe_stop_active" data_type="bool">
     <param name="data_type">bool</param>
-    <param name="min">0</param>
-    <param name="max">1</param>
     <param name="index">0x211A</param>
     <param name="subindex">0x0</param>
@@ -148,6 +148,4 @@
   <state_interface name="toggle_bit" data_type="bool">
     <param name="data_type">bool</param>
-    <param name="min">0</param>
-    <param name="max">1</param>
     <param name="index">0x211B</param>
     <param name="subindex">0x0</param>
@@ -155,6 +153,4 @@
   <state_interface name="load" data_type="int8_t">
     <param name="data_type">int8_t</param>
-    <param name="min">-100</param>
-    <param name="max">100</param>
     <param name="index">0x211C</param>
     <param name="subindex">0x0</param>
@@ -164,6 +160,4 @@
   <state_interface name="velocity" data_type="int16_t">
     <param name="data_type">int16_t</param>
-    <param name="min">-10000</param>
-    <param name="max">10000</param>
     <param name="index">0x211D</param>
     <param name="subindex">0x0</param>
@@ -173,6 +167,4 @@
   <state_interface name="effort" data_type="int16_t">
     <param name="data_type">int16_t</param>
-    <param name="min">-32767</param>
-    <param name="max">32767</param>
     <param name="index">0x211E</param>
     <param name="subindex">0x0</param>
@@ -182,6 +174,4 @@
   <state_interface name="encoder_pulse_counter" data_type="int16_t">
     <param name="data_type">int16_t</param>
-    <param name="min">-32768</param>
-    <param name="max">32767</param>
     <param name="index">0x211F</param>
     <param name="subindex">0x0</param>
@@ -190,6 +180,4 @@
   <state_interface name="fault_warning_code" data_type="uint16_t">
     <param name="data_type">uint16_t</param>
-    <param name="min">0</param>
-    <param name="max">9999</param>
     <param name="index">0x2120</param>
     <param name="subindex">0x0</param>
@@ -197,6 +185,4 @@
   <state_interface name="BDI_level" data_type="uint8_t">
     <param name="data_type">uint8_t</param>
-    <param name="min">0</param>
-    <param name="max">10</param>
     <param name="index">0x2121</param>
     <param name="subindex">0x0</param>
@@ -204,6 +190,4 @@
   <state_interface name="inverter_temperature" data_type="int8_t">
     <param name="data_type">int8_t</param>
-    <param name="min">-60</param>
-    <param name="max">100</param>
     <param name="index">0x2122</param>
     <param name="subindex">0x0</param>
@@ -212,45 +196,21 @@
   <state_interface name="motor_temperature" data_type="int16_t">
     <param name="data_type">int16_t</param>
-    <param name="min">-50</param>
-    <param name="max">200</param>
     <param name="index">0x2123</param>
     <param name="subindex">0x0</param>
   </state_interface>
-  <state_interface name="battery_voltage" data_type="uint16_t">
+  <state_interface name="motor_phase_current" data_type="uint16_t">
     <param name="data_type">uint16_t</param>
-    <param name="min">0</param>
-    <param name="max">65000</param>
-    <param name="index">0x2124</param>
+    <param name="index">0x2126</param>
+    <param name="subindex">0x0</param>
+    <param name="unit">A</param>
+    <param name="from_hw_scaling_factor">0.1</param>
+  </state_interface>
+  <state_interface name="motor_voltage" data_type="uint16_t">
+    <param name="data_type">uint16_t</param>
+    <param name="index">0x2126</param>
     <param name="subindex">0x0</param>
     <param name="unit">V</param>
     <param name="from_hw_scaling_factor">0.01</param>
   </state_interface>
-  <state_interface name="motor_phase_current" data_type="uint16_t">
-    <param name="data_type">uint16_t</param>
-    <param name="min">0</param>
-    <param name="max">29000</param>
-    <param name="index">0x2126</param>
-    <param name="subindex">0x0</param>
-    <param name="unit">A</param>
-    <param name="from_hw_scaling_factor">0.1</param>
-  </state_interface>
-  <state_interface name="motor_voltage" data_type="uint16_t">
-    <param name="data_type">uint16_t</param>
-    <param name="min">0</param>
-    <param name="max">15000</param>
-    <param name="index">0x2126</param>
-    <param name="subindex">0x0</param>
-    <param name="unit">V</param>
-    <param name="from_hw_scaling_factor">0.01</param>
-  </state_interface>
-  <state_interface name="battery_current" data_type="int16_t">
-    <param name="data_type">int16_t</param>
-    <param name="min">-32768</param>
-    <param name="max">32767</param>
-    <param name="index">0x2127</param>
-    <param name="subindex">0x0</param>
-    <param name="unit">A</param>
-    <param name="from_hw_scaling_factor">0.1</param>
-  </state_interface>
 </xacro:macro>
 </robot>
