Commit message: Corrected wheel factors.

File: urdf/mav1500/mav1500_new.ros2_control.xacro (robot description, xacro)
@@ -1,4 +1,5 @@
 <?xml version="1.0"?>
 <robot xmlns:xacro="http://www.ros.org/wiki/xacro">
+<xacro:property name="gear_ratio" value="8.12"/>
 <xacro:macro name="mav1500_ros2_control" params="
               name
@@ -92,5 +93,5 @@
     <param name="subindex">0x0</param>
     <param name="unit">rpm</param>
-    <param name="to_hw_scaling_factor">${inverse_factor * 1.0}</param>
+    <param name="to_hw_scaling_factor">${inverse_factor * 1.0 * gear_ratio}</param>
   </command_interface>
   <command_interface name="torque" data_type="int16_t">
@@ -168,5 +169,5 @@
     <param name="subindex">0x0</param>
     <param name="unit">rpm</param>
-    <param name="from_hw_scaling_factor">${inverse_factor * 1.0}</param>
+    <param name="from_hw_scaling_factor">${inverse_factor * 1.0 * gear_ratio}</param>
   </state_interface>
   <state_interface name="effort" data_type="int16_t">
